File: KICAD/PIC12_BOARD_REV2.sch (KiCad schematic (older format))
At the start: 49 parts, among them J1 USB_B, U1 PIC12F675-IP, U2 LF33_TO220

Commit message: added_schematic
Parts:
- removed VCC1: TestPoint, PCB_ENRICO_FOOTPRINT:TP_EN0, symbol Connector:TestPoint
- C1, C3: value C -> 10uF
- C2: value C -> 10nF
- C4, C5: value C -> 100nF
- U2: value LF33_TO220 -> MIC39100
Connections:
- net DATA+: no longer names the net of J1.3 (D+)
- net DATA-: no longer names the net of J1.2 (D-)
Changed lines of the file:
@@
 encoding utf-8
 Sheet 1 1
-Title ""
-Date ""
-Rev ""
+Title "PIC12_EVALUATION_BOARD"
+Date "2021-11-05"
+Rev "REV_2.0"
 Comp ""
-Comment1 ""
+Comment1 "Designed by ES"
 Comment2 ""
 Comment3 ""
@@
 P 3200 1350
 F 0 "C1" H 3315 1350 50  0000 L CNN
-F 1 "C" H 3315 1305 50  0001 L CNN
+F 1 "10uF" H 3300 1250 50  0000 L CNN
 F 2 "Resistor_SMD:R_0805_2012Metric_Pad1.15x1.40mm_HandSolder" H 3238 1200 50  0001 C CNN
 F 3 "~" H 3200 1350 50  0001 C CNN
@@
 P 4550 1350
 F 0 "C2" H 4665 1350 50  0000 L CNN
-F 1 "C" H 4665 1305 50  0001 L CNN
+F 1 "10nF" H 4650 1250 50  0000 L CNN
 F 2 "Resistor_SMD:R_0805_2012Metric_Pad1.15x1.40mm_HandSolder" H 4588 1200 50  0001 C CNN
 F 3 "~" H 4550 1350 50  0001 C CNN
@@
 P 2600 1000
 F 0 "U2" H 2600 1242 50  0000 C CNN
-F 1 "LF33_TO220" H 2600 1151 50  0000 C CNN
+F 1 "MIC39100" H 2600 1151 50  0000 C CNN
 F 2 "Package_TO_SOT_SMD:SOT-223-3_TabPin2" H 2600 1225 50  0001 C CIN
 F 3 "http://www.st.com/content/ccc/resource/technical/document/datasheet/c4/0e/7e/2a/be/bc/4c/bd/CD00000546.pdf/files/CD00000546.pdf/jcr:content/translations/en.CD00000546.pdf" H 2600 950 50  0001 C CNN
@@
 P 2100 1350
 F 0 "C3" H 2150 1450 50  0000 L CNN
-F 1 "C" H 2215 1305 50  0001 L CNN
+F 1 "10uF" H 2215 1305 50  0000 L CNN
 F 2 "Resistor_SMD:R_0805_2012Metric_Pad1.15x1.40mm_HandSolder" H 2138 1200 50  0001 C CNN
 F 3 "~" H 2100 1350 50  0001 C CNN
@@
 	1    0    0    -1
 $EndComp
-Wire Wire Line
-	5800 3150 5800 3200
 $Comp
 L power:VDD #PWR0107
@@
 P 1800 1350
 F 0 "C4" H 1850 1450 50  0000 L CNN
-F 1 "C" H 1915 1305 50  0001 L CNN
+F 1 "100nF" H 1800 1250 50  0000 L CNN
 F 2 "Resistor_SMD:R_0805_2012Metric_Pad1.15x1.40mm_HandSolder" H 1838 1200 50  0001 C CNN
 F 3 "~" H 1800 1350 50  0001 C CNN
@@
 P 4050 1350
 F 0 "R7" H 4100 1350 50  0000 L CNN
-F 1 "4.7k" H 4120 1305 50  0001 L CNN
+F 1 "4.7k" H 4100 1250 50  0000 L CNN
 F 2 "Resistor_SMD:R_0805_2012Metric_Pad1.15x1.40mm_HandSolder" V 3980 1350 50  0001 C CNN
 F 3 "~" H 4050 1350 50  0001 C CNN
@@
 Wire Wire Line
 	4050 1500 4050 1700
-Text GLabel 1350 1200 2    50   Input ~ 0
-DATA+
-Wire Wire Line
-	1350 1200 1250 1200
-Text GLabel 1350 1300 2    50   Input ~ 0
-DATA-
-Wire Wire Line
-	1350 1300 1250 1300
 $Comp
 L power:+5V #PWR0112
@@
 P 4950 1350
 F 0 "C5" H 5065 1350 50  0000 L CNN
-F 1 "C" H 5065 1305 50  0001 L CNN
+F 1 "100nF" H 5050 1250 50  0000 L CNN
 F 2 "Resistor_SMD:R_0805_2012Metric_Pad1.15x1.40mm_HandSolder" H 4988 1200 50  0001 C CNN
 F 3 "~" H 4950 1350 50  0001 C CNN
@@
 	4950 1700 4550 1700
 Connection ~ 4550 1700
-$Comp
-L Connector:TestPoint VCC1
-U 1 1 5ED2E976
-P 5450 3100
-F 0 "VCC1" H 5508 3218 50  0000 L CNN
-F 1 "TestPoint" H 5508 3127 50  0001 L CNN
-F 2 "PCB_ENRICO_FOOTPRINT:TP_EN0" H 5650 3100 50  0001 C CNN
-F 3 "~" H 5650 3100 50  0001 C CNN
-	1    5450 3100
-	1    0    0    -1
-$EndComp
-Wire Wire Line
-	5450 3100 5450 3200
-Wire Wire Line
-	5450 3200 5800 3200
-Connection ~ 5800 3200
-Wire Wire Line
-	5800 3200 5800 3250
 $Comp
 L Connector:TestPoint GND2
@@
 Wire Wire Line
 	2950 1700 3200 1700
+Wire Wire Line
+	5800 3150 5800 3250
 $EndSCHEMATC
