File: KICAD/PIC12_BOARD_REV2.kicad_pcb (KiCad board)
At the start: 2 copper layers, 70 x 100 mm, 554 parts, among them J1 USB_B, U1 PIC12F675-IP, U2 LF33_TO220

Commit message: open_source_logo
Parts:
- added REF**: OSHW-Symbol_13.4x12mm_SilkScreen, Symbol:OSHW-Symbol_13.4x12mm_SilkScreen, F.Cu at (175.4, 55.1)
